Commit message: feat: definitive URDF - correct link names + joint origins
- Links renamed link1-link6_flange (fixes Gazebo joint matching)
- Joint origins restored from original ROS1 URDF (fixes RViz visuals)
- World link added for MoveIt compatibility
- Inertial tags on all links for Gazebo physics

File: urdf/mycobot_280pi.ros2_control.xacro (robot description, xacro)
@@ -77,94 +77,171 @@
     </plugin>
   </gazebo>
-  <!-- Use simple colored cylinders in Gazebo instead of heavy .dae meshes.
-       This makes Gazebo load instantly while RViz still shows the real meshes.
-       The <gazebo reference> block overrides ONLY what Gazebo sees. -->
   <gazebo reference="base_link">
     <visual>
       <geometry>
-        <cylinder length="0.04" radius="0.06"/>
+        <box>
+          <size>0.1 0.1 0.04</size>
+        </box>
       </geometry>
       <material>
         <ambient>0.1 0.1 0.1 1</ambient>
-        <diffuse>0.1 0.1 0.1 1</diffuse>
-      </material>
-    </visual>
+        <diffuse>0.2 0.2 0.2 1</diffuse>
+      </material>
+    </visual>
+    <collision>
+      <geometry>
+        <box>
+          <size>0.1 0.1 0.04</size>
+        </box>
+      </geometry>
+    </collision>
   </gazebo>
   <gazebo reference="link1">
     <visual>
       <geometry>
-        <cylinder length="0.08" radius="0.04"/>
+        <cylinder>
+          <radius>0.04</radius>
+          <length>0.08</length>
+        </cylinder>
       </geometry>
       <material>
         <ambient>0.5 0.5 0.5 1</ambient>
+        <diffuse>0.6 0.6 0.6 1</diffuse>
+      </material>
+    </visual>
+    <collision>
+      <geometry>
+        <cylinder>
+          <radius>0.04</radius>
+          <length>0.08</length>
+        </cylinder>
+      </geometry>
+    </collision>
+  </gazebo>
+  <gazebo reference="link2">
+    <visual>
+      <geometry>
+        <box>
+          <size>0.11 0.04 0.04</size>
+        </box>
+      </geometry>
+      <material>
+        <ambient>0.8 0.8 0.8 1</ambient>
+        <diffuse>0.9 0.9 0.9 1</diffuse>
+      </material>
+    </visual>
+    <collision>
+      <geometry>
+        <box>
+          <size>0.11 0.04 0.04</size>
+        </box>
+      </geometry>
+    </collision>
+  </gazebo>
+  <gazebo reference="link3">
+    <visual>
+      <geometry>
+        <box>
+          <size>0.096 0.04 0.04</size>
+        </box>
+      </geometry>
+      <material>
+        <ambient>0.8 0.8 0.8 1</ambient>
+        <diffuse>0.9 0.9 0.9 1</diffuse>
+      </material>
+    </visual>
+    <collision>
+      <geometry>
+        <box>
+          <size>0.096 0.04 0.04</size>
+        </box>
+      </geometry>
+    </collision>
+  </gazebo>
+  <gazebo reference="link4">
+    <visual>
+      <geometry>
+        <box>
+          <size>0.096 0.04 0.04</size>
+        </box>
+      </geometry>
+      <material>
+        <ambient>0.4 0.4 0.4 1</ambient>
         <diffuse>0.5 0.5 0.5 1</diffuse>
       </material>
     </visual>
-  </gazebo>
-  <gazebo reference="link2">
-    <visual>
-      <geometry>
-        <box size="0.11 0.04 0.04"/>
-      </geometry>
-      <material>
-        <ambient>0.9 0.9 0.9 1</ambient>
-        <diffuse>0.9 0.9 0.9 1</diffuse>
-      </material>
-    </visual>
-  </gazebo>
-  <gazebo reference="link3">
-    <visual>
-      <geometry>
-        <box size="0.096 0.04 0.04"/>
-      </geometry>
-      <material>
-        <ambient>0.9 0.9 0.9 1</ambient>
-        <diffuse>0.9 0.9 0.9 1</diffuse>
-      </material>
-    </visual>
-  </gazebo>
-  <gazebo reference="link4">
-    <visual>
-      <geometry>
-        <box size="0.096 0.04 0.04"/>
-      </geometry>
-      <material>
-        <ambient>0.5 0.5 0.5 1</ambient>
+    <collision>
+      <geometry>
+        <box>
+          <size>0.096 0.04 0.04</size>
+        </box>
+      </geometry>
+    </collision>
+  </gazebo>
+  <gazebo reference="link5">
+    <visual>
+      <geometry>
+        <cylinder>
+          <radius>0.03</radius>
+          <length>0.04</length>
+        </cylinder>
+      </geometry>
+      <material>
+        <ambient>0.1 0.1 0.1 1</ambient>
+        <diffuse>0.2 0.2 0.2 1</diffuse>
+      </material>
+    </visual>
+    <collision>
+      <geometry>
+        <cylinder>
+          <radius>0.03</radius>
+          <length>0.04</length>
+        </cylinder>
+      </geometry>
+    </collision>
+  </gazebo>
+  <gazebo reference="link6">
+    <visual>
+      <geometry>
+        <cylinder>
+          <radius>0.03</radius>
+          <length>0.04</length>
+        </cylinder>
+      </geometry>
+      <material>
+        <ambient>0.4 0.4 0.4 1</ambient>
         <diffuse>0.5 0.5 0.5 1</diffuse>
       </material>
     </visual>
-  </gazebo>
-  <gazebo reference="link5">
-    <visual>
-      <geometry>
-        <cylinder length="0.04" radius="0.03"/>
+    <collision>
+      <geometry>
+        <cylinder>
+          <radius>0.03</radius>
+          <length>0.04</length>
+        </cylinder>
+      </geometry>
+    </collision>
+  </gazebo>
+  <gazebo reference="link6_flange">
+    <visual>
+      <geometry>
+        <cylinder>
+          <radius>0.025</radius>
+          <length>0.02</length>
+        </cylinder>
       </geometry>
       <material>
         <ambient>0.1 0.1 0.1 1</ambient>
-        <diffuse>0.1 0.1 0.1 1</diffuse>
-      </material>
-    </visual>
-  </gazebo>
-  <gazebo reference="link6">
-    <visual>
-      <geometry>
-        <cylinder length="0.04" radius="0.03"/>
-      </geometry>
-      <material>
-        <ambient>0.5 0.5 0.5 1</ambient>
-        <diffuse>0.5 0.5 0.5 1</diffuse>
-      </material>
-    </visual>
-  </gazebo>
-  <gazebo reference="link6_flange">
-    <visual>
-      <geometry>
-        <cylinder length="0.02" radius="0.025"/>
-      </geometry>
-      <material>
-        <ambient>0.1 0.1 0.1 1</ambient>
-        <diffuse>0.1 0.1 0.1 1</diffuse>
-      </material>
-    </visual>
+        <diffuse>0.2 0.2 0.2 1</diffuse>
+      </material>
+    </visual>
+    <collision>
+      <geometry>
+        <cylinder>
+          <radius>0.025</radius>
+          <length>0.02</length>
+        </cylinder>
+      </geometry>
+    </collision>
   </gazebo>
 </robot>

File: urdf/mycobot_280pi.urdf.xacro (robot description, xacro)
@@ -1,5 +1,12 @@
-<?xml version="1.1"?>
-<robot  xmlns:xacro="http://www.ros.org/wiki/xacro" name="firefighter" >
-<xacro:property name="width" value=".2" />
+<?xml version="1.0"?>
+<robot xmlns:xacro="http://www.ros.org/wiki/xacro" name="mycobot_280pi">
+  <xacro:property name="width" value=".2"/>
+  <xacro:include filename="$(find mycobot_280pi_description)/urdf/mycobot_280pi.ros2_control.xacro"/>
+  <link name="world"/>
+  <joint name="world_to_base" type="fixed">
+    <parent link="world"/>
+    <child link="base_link"/>
+    <origin xyz="0 0 0" rpy="0 0 0"/>
+  </joint>
   <link name="base_link">
     <visual>
@@ -7,5 +14,5 @@
         <mesh filename="package://mycobot_280pi_description/meshes/visual/G_base.dae"/>
       </geometry>
-      <origin xyz = "0.0 0 -0.03" rpy = "0 0 1.5708"/>
+      <origin xyz="0.0 0 -0.03" rpy="0 0 1.5708"/>
     </visual>
     <collision>
@@ -13,163 +20,197 @@
         <mesh filename="package://mycobot_280pi_description/meshes/visual/G_base.dae"/>
       </geometry>
-      <origin xyz = "0.0 0 -0.03" rpy = "0 0 1.5708"/>
-    </collision>
-  </link>
-  <link name="joint1">
-    <visual>
-      <geometry>
-	     <!--- 0.0 0 -0.04  1.5708 3.14159-->
-       <mesh filename="package://mycobot_280pi_description/meshes/visual/joint1_pi.dae"/>
-      </geometry>
-    <origin xyz = "0.0 0 0 " rpy = " 0 0 0"/>
-    </visual>
-    <collision>
-      <geometry>
-	     <!--- 0.0 0 -0.04  1.5708 3.14159-->
-       <mesh filename="package://mycobot_280pi_description/meshes/visual/joint1_pi.dae"/>
-      </geometry>
-    <origin xyz = "0.0 0 0 " rpy = " 0 0 0"/>
-    </collision>
-  </link>
-  <link name="joint2">
-    <visual>
-      <geometry>
-       <mesh filename="package://mycobot_280pi_description/meshes/visual/joint2.dae"/>
-      </geometry>
-    <origin xyz = "0.0 0 -0.06096 " rpy = " 0 0 -1.5708"/>
-    </visual>
-      <collision>
-      <geometry>
-       <mesh filename="package://mycobot_280pi_description/meshes/visual/joint2.dae"/>
-      </geometry>
-    <origin xyz = "0.0 0 -0.06096 " rpy = " 0 0 -1.5708"/>
-    </collision>
-  </link>
-  <link name="joint3">
-    <visual>
-      <geometry>
-       <mesh filename="package://mycobot_280pi_description/meshes/visual/joint3.dae"/>
-      </geometry>
-    <origin xyz = "0.0 0 0.03256 " rpy = " 0 -1.5708 0"/>
-    </visual>
-      <collision>
-        <geometry>
-       <mesh filename="package://mycobot_280pi_description/meshes/visual/joint3.dae"/>
-      </geometry>
-    <origin xyz = "0.0 0 0.03256 " rpy = " 0 -1.5708 0"/>
-    </collision>
-  </link>
-  <link name="joint4">
-    <visual>
-      <geometry>
-       <!--- 0.0 0 -0.04 -->
-       <mesh filename="package://mycobot_280pi_description/meshes/visual/joint4.dae"/>
-      </geometry>
-    <origin xyz = "0.0 0 0.03056 " rpy = " 0 -1.5708 0"/>
-    </visual>
-      <collision>
-      <geometry>
-       <!--- 0.0 0 -0.04 -->
-       <mesh filename="package://mycobot_280pi_description/meshes/visual/joint4.dae"/>
-      </geometry>
-    <origin xyz = "0.0 0 0.03056 " rpy = " 0 -1.5708 0"/>
-    </collision>
-  </link>
-<link name="joint5">
-    <visual>
-      <geometry>
-       <!--- 0.0 0 -0.04 -->
-       <mesh filename="package://mycobot_280pi_description/meshes/visual/joint5.dae"/>
-      </geometry>
-    <origin xyz = "0.0 -0.001 -0.0345 " rpy = " 0 -1.5708 1.5708"/>
-    </visual>
-      <collision>
-      <geometry>
-       <!--- 0.0 0 -0.04 -->
-       <mesh filename="package://mycobot_280pi_description/meshes/visual/joint5.dae"/>
-      </geometry>
-    <origin xyz = "0.0 -0.001 -0.0345 " rpy = " 0 -1.5708 1.5708"/>
-    </collision>
-  </link>
-  <link name="joint6">
-    <visual>
-      <geometry>
-       <!--- 0.0 0 -0.04 -->
-       <mesh filename="package://mycobot_280pi_description/meshes/visual/joint6.dae"/>
-      </geometry>
-    <origin xyz = "0 0.00 -0.038 " rpy = " 0 0 0"/>
-    </visual>
-      <collision>
-      <geometry>
-       <!--- 0.0 0 -0.04 -->
-       <mesh filename="package://mycobot_280pi_description/meshes/visual/joint6.dae"/>
-      </geometry>
-    <origin xyz = "0 0.00 -0.038 " rpy = " 0 0 0"/>
-    </collision>
-  </link>
-  <link name="joint6_flange">
-    <visual>
-      <geometry>
-       <!--- 0.0 0 -0.04 -->
-       <mesh filename="package://mycobot_280pi_description/meshes/visual/joint7.dae"/>
-      </geometry>
-    <origin xyz = "0.0 0 -0.012 " rpy = " 0 0 0"/>
-    </visual>
-      <collision>
-      <geometry>
-       <!--- 0.0 0 -0.04 -->
-       <mesh filename="package://mycobot_280pi_description/meshes/visual/joint7.dae"/>
-      </geometry>
-    <origin xyz = "0.0 0 -0.012 " rpy = " 0 0 0"/>
-    </collision>
-  </link>
-  <joint name="g_base_to_joint1" type="fixed">
-    <axis xyz="0 0 0"/>
-    <limit effort = "1000.0" lower = "-3.14" upper = "3.14159" velocity = "0"/>
+      <origin xyz="0.0 0 -0.03" rpy="0 0 1.5708"/>
+    </collision>
+    <inertial>
+      <origin xyz="0 0 0" rpy="0 0 0"/>
+      <mass value="1.0"/>
+      <inertia ixx="0.005" ixy="0" ixz="0" iyy="0.005" iyz="0" izz="0.003"/>
+    </inertial>
+  </link>
+  <link name="link1">
+    <visual>
+      <geometry>
+        <mesh filename="package://mycobot_280pi_description/meshes/visual/joint1_pi.dae"/>
+      </geometry>
+      <origin xyz="0.0 0.0 0.0" rpy="0 0 0"/>
+    </visual>
+    <collision>
+      <geometry>
+        <mesh filename="package://mycobot_280pi_description/meshes/visual/joint1_pi.dae"/>
+      </geometry>
+      <origin xyz="0.0 0.0 0.0" rpy="0 0 0"/>
+    </collision>
+    <inertial>
+      <origin xyz="0 0 0" rpy="0 0 0"/>
+      <mass value="0.24"/>
+      <inertia ixx="0.0002" ixy="0" ixz="0" iyy="0.0002" iyz="0" izz="0.0001"/>
+    </inertial>
+  </link>
+  <link name="link2">
+    <visual>
+      <geometry>
+        <mesh filename="package://mycobot_280pi_description/meshes/visual/joint2.dae"/>
+      </geometry>
+      <origin xyz="0.0 0.0 -0.06096" rpy="0 0 -1.5708"/>
+    </visual>
+    <collision>
+      <geometry>
+        <mesh filename="package://mycobot_280pi_description/meshes/visual/joint2.dae"/>
+      </geometry>
+      <origin xyz="0.0 0.0 -0.06096" rpy="0 0 -1.5708"/>
+    </collision>
+    <inertial>
+      <origin xyz="0 0 0" rpy="0 0 0"/>
+      <mass value="0.22"/>
+      <inertia ixx="0.0003" ixy="0" ixz="0" iyy="0.0003" iyz="0" izz="0.00005"/>
+    </inertial>
+  </link>
+  <link name="link3">
+    <visual>
+      <geometry>
+        <mesh filename="package://mycobot_280pi_description/meshes/visual/joint3.dae"/>
+      </geometry>
+      <origin xyz="0.0 0.0 0.03256" rpy="0 -1.5708 0"/>
+    </visual>
+    <collision>
+      <geometry>
+        <mesh filename="package://mycobot_280pi_description/meshes/visual/joint3.dae"/>
+      </geometry>
+      <origin xyz="0.0 0.0 0.03256" rpy="0 -1.5708 0"/>
+    </collision>
+    <inertial>
+      <origin xyz="0 0 0" rpy="0 0 0"/>
+      <mass value="0.15"/>
+      <inertia ixx="0.0001" ixy="0" ixz="0" iyy="0.0002" iyz="0" izz="0.00005"/>
+    </inertial>
+  </link>
+  <link name="link4">
+    <visual>
+      <geometry>
+        <mesh filename="package://mycobot_280pi_description/meshes/visual/joint4.dae"/>
+      </geometry>
+      <origin xyz="0.0 0.0 0.03056" rpy="0 -1.5708 0"/>
+    </visual>
+    <collision>
+      <geometry>
+        <mesh filename="package://mycobot_280pi_description/meshes/visual/joint4.dae"/>
+      </geometry>
+      <origin xyz="0.0 0.0 0.03056" rpy="0 -1.5708 0"/>
+    </collision>
+    <inertial>
+      <origin xyz="0 0 0" rpy="0 0 0"/>
+      <mass value="0.13"/>
+      <inertia ixx="0.00008" ixy="0" ixz="0" iyy="0.0001" iyz="0" izz="0.00003"/>
+    </inertial>
+  </link>
+  <link name="link5">
+    <visual>
+      <geometry>
+        <mesh filename="package://mycobot_280pi_description/meshes/visual/joint5.dae"/>
+      </geometry>
+      <origin xyz="0.0 -0.001 -0.0345" rpy="0 -1.5708 1.5708"/>
+    </visual>
+    <collision>
+      <geometry>
+        <mesh filename="package://mycobot_280pi_description/meshes/visual/joint5.dae"/>
+      </geometry>
+      <origin xyz="0.0 -0.001 -0.0345" rpy="0 -1.5708 1.5708"/>
+    </collision>
+    <inertial>
+      <origin xyz="0 0 0" rpy="0 0 0"/>
+      <mass value="0.10"/>
+      <inertia ixx="0.00005" ixy="0" ixz="0" iyy="0.00005" iyz="0" izz="0.00003"/>
+    </inertial>
+  </link>
+  <link name="link6">
+    <visual>
+      <geometry>
+        <mesh filename="package://mycobot_280pi_description/meshes/visual/joint6.dae"/>
+      </geometry>
+      <origin xyz="0 0.00 -0.038" rpy="0 0 0"/>
+    </visual>
+    <collision>
+      <geometry>
+        <mesh filename="package://mycobot_280pi_description/meshes/visual/joint6.dae"/>
+      </geometry>
+      <origin xyz="0 0.00 -0.038" rpy="0 0 0"/>
+    </collision>
+    <inertial>
+      <origin xyz="0 0 0" rpy="0 0 0"/>
+      <mass value="0.08"/>
+      <inertia ixx="0.00003" ixy="0" ixz="0" iyy="0.00003" iyz="0" izz="0.00002"/>
+    </inertial>
+  </link>
+  <link name="link6_flange">
+    <visual>
+      <geometry>
+        <mesh filename="package://mycobot_280pi_description/meshes/visual/joint7.dae"/>
+      </geometry>
+      <origin xyz="0.0 0.0 -0.012" rpy="0 0 0"/>
+    </visual>
+    <collision>
+      <geometry>
+        <mesh filename="package://mycobot_280pi_description/meshes/visual/joint7.dae"/>
+      </geometry>
+      <origin xyz="0.0 0.0 -0.012" rpy="0 0 0"/>
+    </collision>
+    <inertial>
+      <origin xyz="0 0 0" rpy="0 0 0"/>
+      <mass value="0.05"/>
+      <inertia ixx="0.00001" ixy="0" ixz="0" iyy="0.00001" iyz="0" izz="0.00001"/>
+    </inertial>
+  </link>
+  <joint name="base_to_link1" type="fixed">
     <parent link="base_link"/>
-    <child link="joint1"/>
-    <origin xyz= "0 0 0" rpy = "0 0 0"/>
+    <child link="link1"/>
+    <origin xyz="0 0 0" rpy="0 0 0"/>
   </joint>
   <joint name="joint2_to_joint1" type="revolute">
     <axis xyz="0 0 1"/>
-    <limit effort = "1000.0" lower = "-2.9321" upper = "2.9321" velocity = "0"/>
-    <parent link="joint1"/>
-    <child link="joint2"/>
-    <origin xyz= "0 0 0.13956" rpy = "0 0 0"/>
+    <limit effort="1000.0" lower="-2.9321" upper="2.9321" velocity="2.0"/>
+    <parent link="link1"/>
+    <child link="link2"/>
+    <origin xyz="0 0 0.13956" rpy="0 1.5708 -1.5708"/>
+    <dynamics damping="0.1" friction="0.1"/>
   </joint>
   <joint name="joint3_to_joint2" type="revolute">
     <axis xyz="0 0 1"/>
-    <limit effort = "1000.0" lower = "-2.4434" upper = "2.4434" velocity = "0"/>
-    <parent link="joint2"/>
-    <child link="joint3"/>
-    <origin xyz= "0 0 -0.001" rpy = "0 1.5708 -1.5708"/>
+    <limit effort="1000.0" lower="-2.4434" upper="2.4434" velocity="2.0"/>
+    <parent link="link2"/>
+    <child link="link3"/>
+    <origin xyz="-0.1104 0 0" rpy="0 0 0"/>
+    <dynamics damping="0.1" friction="0.1"/>
   </joint>
   <joint name="joint4_to_joint3" type="revolute">
-    <axis xyz=" 0 0 1"/>
-    <limit effort = "1000.0" lower = "-2.6179" upper = "2.6179" velocity = "0"/>
-    <parent link="joint3"/>
-    <child link="joint4"/>
-    <origin xyz= "  -0.1104 0 0   " rpy = "0 0 0"/>
+    <axis xyz="0 0 1"/>
+    <limit effort="1000.0" lower="-2.6179" upper="2.6179" velocity="2.0"/>
+    <parent link="link3"/>
+    <child link="link4"/>
+    <origin xyz="-0.096 0 0.06462" rpy="0 0 -1.5708"/>
+    <dynamics damping="0.1" friction="0.1"/>
   </joint>
   <joint name="joint5_to_joint4" type="revolute">
-    <axis xyz=" 0 0 1"/>
-    <limit effort = "1000.0" lower = "-2.6179" upper = "2.6179" velocity = "0"/>
-    <parent link="joint4"/>
-    <child link="joint5"/>
-    <origin xyz= "-0.096 0 0.06462" rpy = "0 0 -1.5708"/>
+    <axis xyz="0 0 1"/>
+    <limit effort="1000.0" lower="-2.6179" upper="2.6179" velocity="2.0"/>
+    <parent link="link4"/>
+    <child link="link5"/>
+    <origin xyz="0 -0.07318 -0.001" rpy="1.5708 -1.5708 0"/>
+    <dynamics damping="0.1" friction="0.1"/>
   </joint>
   <joint name="joint6_to_joint5" type="revolute">
     <axis xyz="0 0 1"/>
-    <limit effort = "1000.0" lower = "-2.7052" upper = "2.7925" velocity = "0"/>
-    <parent link="joint5"/>
-    <child link="joint6"/>
-    <origin xyz= "0 -0.07318 -0.001" rpy = "1.5708 -1.5708 0"/>
+    <limit effort="1000.0" lower="-2.7052" upper="2.7925" velocity="2.0"/>
+    <parent link="link5"/>
+    <child link="link6"/>
+    <origin xyz="0 0.0456 0" rpy="-1.5708 0 0"/>
+    <dynamics damping="0.1" friction="0.1"/>
   </joint>
   <joint name="joint6output_to_joint6" type="revolute">
     <axis xyz="0 0 1"/>
-    <limit effort = "1000.0" lower = "-3.14159" upper = "3.14159" velocity = "0"/>
-    <parent link="joint6"/>
-    <child link="joint6_flange"/>
-    <origin xyz= "0 0.0456 0" rpy = "-1.5708 0 0"/>
+    <limit effort="1000.0" lower="-3.14159" upper="3.14159" velocity="2.0"/>
+    <parent link="link6"/>
+    <child link="link6_flange"/>
+    <origin xyz="0 0 0" rpy="0 0 0"/>
+    <dynamics damping="0.1" friction="0.1"/>
   </joint>
 </robot>
