Commit message: fix: revert to original link naming (joint1-joint6)
- Restored original Elephant Robotics link names for correct mesh alignment
- Kept base_link and world link for ROS 2 convention
- Restored original joint origins from ROS1 URDF
- Fixed XML declaration to version 1.1 to prevent gazebo_ros2_control parser crash
- Added proper SDF geometry for Gazebo visuals

File: urdf/mycobot_280pi.ros2_control.xacro (robot description, xacro)
@@ -75,4 +75,6 @@
     <plugin name="gazebo_ros2_control" filename="libgazebo_ros2_control.so">
       <parameters>$(find mycobot_280pi_gazebo)/config/controllers.yaml</parameters>
+      <robot_param>robot_description</robot_param>
+      <robot_param_node>robot_state_publisher</robot_param_node>
     </plugin>
   </gazebo>
@@ -97,5 +99,5 @@
     </collision>
   </gazebo>
-  <gazebo reference="link1">
+  <gazebo reference="joint1">
     <visual>
       <geometry>
@@ -119,5 +121,5 @@
     </collision>
   </gazebo>
-  <gazebo reference="link2">
+  <gazebo reference="joint2">
     <visual>
       <geometry>
@@ -139,5 +141,5 @@
     </collision>
   </gazebo>
-  <gazebo reference="link3">
+  <gazebo reference="joint3">
     <visual>
       <geometry>
@@ -159,5 +161,5 @@
     </collision>
   </gazebo>
-  <gazebo reference="link4">
+  <gazebo reference="joint4">
     <visual>
       <geometry>
@@ -179,5 +181,5 @@
     </collision>
   </gazebo>
-  <gazebo reference="link5">
+  <gazebo reference="joint5">
     <visual>
       <geometry>
@@ -201,5 +203,5 @@
     </collision>
   </gazebo>
-  <gazebo reference="link6">
+  <gazebo reference="joint6">
     <visual>
       <geometry>
@@ -223,5 +225,5 @@
     </collision>
   </gazebo>
-  <gazebo reference="link6_flange">
+  <gazebo reference="joint6_flange">
     <visual>
       <geometry>

File: urdf/mycobot_280pi.urdf.xacro (robot description, xacro)
@@ -1,6 +1,7 @@
-<?xml version="1.0"?>
+<?xml version="1.1"?>
 <robot xmlns:xacro="http://www.ros.org/wiki/xacro" name="mycobot_280pi">
   <xacro:property name="width" value=".2"/>
   <xacro:include filename="$(find mycobot_280pi_description)/urdf/mycobot_280pi.ros2_control.xacro"/>
+  <!-- World link required by MoveIt and KDL -->
   <link name="world"/>
   <joint name="world_to_base" type="fixed">
@@ -9,4 +10,5 @@
     <origin xyz="0 0 0" rpy="0 0 0"/>
   </joint>
+  <!-- base_link replaces g_base — same geometry, ROS 2 naming convention -->
   <link name="base_link">
     <visual>
@@ -28,5 +30,6 @@
     </inertial>
   </link>
-  <link name="link1">
+  <!-- Original link names from Elephant Robotics restored -->
+  <link name="joint1">
     <visual>
       <geometry>
@@ -47,5 +50,5 @@
     </inertial>
   </link>
-  <link name="link2">
+  <link name="joint2">
     <visual>
       <geometry>
@@ -66,5 +69,5 @@
     </inertial>
   </link>
-  <link name="link3">
+  <link name="joint3">
     <visual>
       <geometry>
@@ -85,5 +88,5 @@
     </inertial>
   </link>
-  <link name="link4">
+  <link name="joint4">
     <visual>
       <geometry>
@@ -104,5 +107,5 @@
     </inertial>
   </link>
-  <link name="link5">
+  <link name="joint5">
     <visual>
       <geometry>
@@ -123,5 +126,5 @@
     </inertial>
   </link>
-  <link name="link6">
+  <link name="joint6">
     <visual>
       <geometry>
@@ -142,5 +145,5 @@
     </inertial>
   </link>
-  <link name="link6_flange">
+  <link name="joint6_flange">
     <visual>
       <geometry>
@@ -161,7 +164,9 @@
     </inertial>
   </link>
-  <joint name="base_to_link1" type="fixed">
+  <!-- ===================== JOINTS ===================== -->
+  <!-- Exact original joint origins from Elephant Robotics ROS1 URDF -->
+  <joint name="base_to_joint1" type="fixed">
     <parent link="base_link"/>
-    <child link="link1"/>
+    <child link="joint1"/>
     <origin xyz="0 0 0" rpy="0 0 0"/>
   </joint>
@@ -169,7 +174,7 @@
     <axis xyz="0 0 1"/>
     <limit effort="1000.0" lower="-2.9321" upper="2.9321" velocity="2.0"/>
-    <parent link="link1"/>
-    <child link="link2"/>
-    <origin xyz="0 0 0.13956" rpy="0 1.5708 -1.5708"/>
+    <parent link="joint1"/>
+    <child link="joint2"/>
+    <origin xyz="0 0 0.13956" rpy="0 0 0"/>
     <dynamics damping="0.1" friction="0.1"/>
   </joint>
@@ -177,40 +182,40 @@
     <axis xyz="0 0 1"/>
     <limit effort="1000.0" lower="-2.4434" upper="2.4434" velocity="2.0"/>
-    <parent link="link2"/>
-    <child link="link3"/>
+    <parent link="joint2"/>
+    <child link="joint3"/>
+    <origin xyz="0 0 -0.001" rpy="0 1.5708 -1.5708"/>
+    <dynamics damping="0.1" friction="0.1"/>
+  </joint>
+  <joint name="joint4_to_joint3" type="revolute">
+    <axis xyz="0 0 1"/>
+    <limit effort="1000.0" lower="-2.6179" upper="2.6179" velocity="2.0"/>
+    <parent link="joint3"/>
+    <child link="joint4"/>
     <origin xyz="-0.1104 0 0" rpy="0 0 0"/>
     <dynamics damping="0.1" friction="0.1"/>
   </joint>
-  <joint name="joint4_to_joint3" type="revolute">
+  <joint name="joint5_to_joint4" type="revolute">
     <axis xyz="0 0 1"/>
     <limit effort="1000.0" lower="-2.6179" upper="2.6179" velocity="2.0"/>
-    <parent link="link3"/>
-    <child link="link4"/>
+    <parent link="joint4"/>
+    <child link="joint5"/>
     <origin xyz="-0.096 0 0.06462" rpy="0 0 -1.5708"/>
     <dynamics damping="0.1" friction="0.1"/>
   </joint>
-  <joint name="joint5_to_joint4" type="revolute">
-    <axis xyz="0 0 1"/>
-    <limit effort="1000.0" lower="-2.6179" upper="2.6179" velocity="2.0"/>
-    <parent link="link4"/>
-    <child link="link5"/>
+  <joint name="joint6_to_joint5" type="revolute">
+    <axis xyz="0 0 1"/>
+    <limit effort="1000.0" lower="-2.7052" upper="2.7925" velocity="2.0"/>
+    <parent link="joint5"/>
+    <child link="joint6"/>
     <origin xyz="0 -0.07318 -0.001" rpy="1.5708 -1.5708 0"/>
     <dynamics damping="0.1" friction="0.1"/>
   </joint>
-  <joint name="joint6_to_joint5" type="revolute">
-    <axis xyz="0 0 1"/>
-    <limit effort="1000.0" lower="-2.7052" upper="2.7925" velocity="2.0"/>
-    <parent link="link5"/>
-    <child link="link6"/>
+  <joint name="joint6output_to_joint6" type="revolute">
+    <axis xyz="0 0 1"/>
+    <limit effort="1000.0" lower="-3.14159" upper="3.14159" velocity="2.0"/>
+    <parent link="joint6"/>
+    <child link="joint6_flange"/>
     <origin xyz="0 0.0456 0" rpy="-1.5708 0 0"/>
     <dynamics damping="0.1" friction="0.1"/>
   </joint>
-  <joint name="joint6output_to_joint6" type="revolute">
-    <axis xyz="0 0 1"/>
-    <limit effort="1000.0" lower="-3.14159" upper="3.14159" velocity="2.0"/>
-    <parent link="link6"/>
-    <child link="link6_flange"/>
-    <origin xyz="0 0 0" rpy="0 0 0"/>
-    <dynamics damping="0.1" friction="0.1"/>
-  </joint>
 </robot>

Commit message: feat: add use_sim xacro argument for sim/real robot switch
- Hardware plugin switches between GazeboSystem and MyCobotHardwareInterface
- Gazebo visual overrides wrapped in xacro:if use_sim block
- Gazebo plugin wrapped in xacro:if use_sim block
- Joint declarations identical for both modes
- Single URDF file works for simulation and real hardware

File: urdf/mycobot_280pi.ros2_control.xacro (robot description, xacro)
@@ -1,8 +1,27 @@
 <?xml version="1.0"?>
 <robot xmlns:xacro="http://www.ros.org/wiki/xacro">
-  <ros2_control name="mycobot_280pi_gazebo" type="system">
+  <!-- ================================================================
+       SIMULATION vs REAL ROBOT SWITCH
+       use_sim:=true  → Gazebo physics engine is the hardware
+       use_sim:=false → Real myCobot 280 Pi connected via USB
+       Everything below the hardware block is identical for both.
+       This is the ros2_control abstraction in action — controllers
+       don't know or care what's underneath them.
+       ================================================================ -->
+  <xacro:arg name="use_sim" default="true"/>
+  <ros2_control name="mycobot_280pi" type="system">
     <hardware>
-      <plugin>gazebo_ros2_control/GazeboSystem</plugin>
+      <!-- SIMULATION MODE -->
+      <xacro:if value="$(arg use_sim)">
+        <plugin>gazebo_ros2_control/GazeboSystem</plugin>
+      </xacro:if>
+      <!-- REAL ROBOT MODE -->
+      <xacro:unless value="$(arg use_sim)">
+        <plugin>mycobot_hardware_interface/MyCobotHardwareInterface</plugin>
+        <param name="port">/dev/ttyUSB0</param>
+        <param name="baud_rate">115200</param>
+      </xacro:unless>
     </hardware>
+    <!-- Joint declarations are identical for sim and real -->
     <joint name="joint2_to_joint1">
       <command_interface name="position">
@@ -72,178 +91,130 @@
     </joint>
   </ros2_control>
-  <gazebo>
-    <plugin name="gazebo_ros2_control" filename="libgazebo_ros2_control.so">
-      <parameters>$(find mycobot_280pi_gazebo)/config/controllers.yaml</parameters>
-      <robot_param>robot_description</robot_param>
-      <robot_param_node>robot_state_publisher</robot_param_node>
-    </plugin>
-  </gazebo>
-  <gazebo reference="base_link">
-    <visual>
-      <geometry>
-        <box>
-          <size>0.1 0.1 0.04</size>
-        </box>
-      </geometry>
-      <material>
-        <ambient>0.1 0.1 0.1 1</ambient>
-        <diffuse>0.2 0.2 0.2 1</diffuse>
-      </material>
-    </visual>
-    <collision>
-      <geometry>
-        <box>
-          <size>0.1 0.1 0.04</size>
-        </box>
-      </geometry>
-    </collision>
-  </gazebo>
-  <gazebo reference="joint1">
-    <visual>
-      <geometry>
-        <cylinder>
-          <radius>0.04</radius>
-          <length>0.08</length>
-        </cylinder>
-      </geometry>
-      <material>
-        <ambient>0.5 0.5 0.5 1</ambient>
-        <diffuse>0.6 0.6 0.6 1</diffuse>
-      </material>
-    </visual>
-    <collision>
-      <geometry>
-        <cylinder>
-          <radius>0.04</radius>
-          <length>0.08</length>
-        </cylinder>
-      </geometry>
-    </collision>
-  </gazebo>
-  <gazebo reference="joint2">
-    <visual>
-      <geometry>
-        <box>
-          <size>0.11 0.04 0.04</size>
-        </box>
-      </geometry>
-      <material>
-        <ambient>0.8 0.8 0.8 1</ambient>
-        <diffuse>0.9 0.9 0.9 1</diffuse>
-      </material>
-    </visual>
-    <collision>
-      <geometry>
-        <box>
-          <size>0.11 0.04 0.04</size>
-        </box>
-      </geometry>
-    </collision>
-  </gazebo>
-  <gazebo reference="joint3">
-    <visual>
-      <geometry>
-        <box>
-          <size>0.096 0.04 0.04</size>
-        </box>
-      </geometry>
-      <material>
-        <ambient>0.8 0.8 0.8 1</ambient>
-        <diffuse>0.9 0.9 0.9 1</diffuse>
-      </material>
-    </visual>
-    <collision>
-      <geometry>
-        <box>
-          <size>0.096 0.04 0.04</size>
-        </box>
-      </geometry>
-    </collision>
-  </gazebo>
-  <gazebo reference="joint4">
-    <visual>
-      <geometry>
-        <box>
-          <size>0.096 0.04 0.04</size>
-        </box>
-      </geometry>
-      <material>
-        <ambient>0.4 0.4 0.4 1</ambient>
-        <diffuse>0.5 0.5 0.5 1</diffuse>
-      </material>
-    </visual>
-    <collision>
-      <geometry>
-        <box>
-          <size>0.096 0.04 0.04</size>
-        </box>
-      </geometry>
-    </collision>
-  </gazebo>
-  <gazebo reference="joint5">
-    <visual>
-      <geometry>
-        <cylinder>
-          <radius>0.03</radius>
-          <length>0.04</length>
-        </cylinder>
-      </geometry>
-      <material>
-        <ambient>0.1 0.1 0.1 1</ambient>
-        <diffuse>0.2 0.2 0.2 1</diffuse>
-      </material>
-    </visual>
-    <collision>
-      <geometry>
-        <cylinder>
-          <radius>0.03</radius>
-          <length>0.04</length>
-        </cylinder>
-      </geometry>
-    </collision>
-  </gazebo>
-  <gazebo reference="joint6">
-    <visual>
-      <geometry>
-        <cylinder>
-          <radius>0.03</radius>
-          <length>0.04</length>
-        </cylinder>
-      </geometry>
-      <material>
-        <ambient>0.4 0.4 0.4 1</ambient>
-        <diffuse>0.5 0.5 0.5 1</diffuse>
-      </material>
-    </visual>
-    <collision>
-      <geometry>
-        <cylinder>
-          <radius>0.03</radius>
-          <length>0.04</length>
-        </cylinder>
-      </geometry>
-    </collision>
-  </gazebo>
-  <gazebo reference="joint6_flange">
-    <visual>
-      <geometry>
-        <cylinder>
-          <radius>0.025</radius>
-          <length>0.02</length>
-        </cylinder>
-      </geometry>
-      <material>
-        <ambient>0.1 0.1 0.1 1</ambient>
-        <diffuse>0.2 0.2 0.2 1</diffuse>
-      </material>
-    </visual>
-    <collision>
-      <geometry>
-        <cylinder>
-          <radius>0.025</radius>
-          <length>0.02</length>
-        </cylinder>
-      </geometry>
-    </collision>
-  </gazebo>
+  <!-- Gazebo plugin — only needed in simulation mode -->
+  <xacro:if value="$(arg use_sim)">
+    <gazebo>
+      <plugin name="gazebo_ros2_control" filename="libgazebo_ros2_control.so">
+        <parameters>$(find mycobot_280pi_gazebo)/config/controllers.yaml</parameters>
+        <robot_param>robot_description</robot_param>
+        <robot_param_node>robot_state_publisher</robot_param_node>
+      </plugin>
+    </gazebo>
+  </xacro:if>
+  <!-- Gazebo visual overrides — only in simulation -->
+  <xacro:if value="$(arg use_sim)">
+    <gazebo reference="base_link">
+      <visual>
+        <geometry>
+          <box><size>0.1 0.1 0.04</size></box>
+        </geometry>
+        <material>
+          <ambient>0.1 0.1 0.1 1</ambient>
+          <diffuse>0.2 0.2 0.2 1</diffuse>
+        </material>
+      </visual>
+      <collision>
+        <geometry><box><size>0.1 0.1 0.04</size></box></geometry>
+      </collision>
+    </gazebo>
+    <gazebo reference="joint1">
+      <visual>
+        <geometry>
+          <cylinder><radius>0.04</radius><length>0.08</length></cylinder>
+        </geometry>
+        <material>
+          <ambient>0.5 0.5 0.5 1</ambient>
+          <diffuse>0.6 0.6 0.6 1</diffuse>
+        </material>
+      </visual>
+      <collision>
+        <geometry>
+          <cylinder><radius>0.04</radius><length>0.08</length></cylinder>
+        </geometry>
+      </collision>
+    </gazebo>
+    <gazebo reference="joint2">
+      <visual>
+        <geometry><box><size>0.11 0.04 0.04</size></box></geometry>
+        <material>
+          <ambient>0.8 0.8 0.8 1</ambient>
+          <diffuse>0.9 0.9 0.9 1</diffuse>
+        </material>
+      </visual>
+      <collision>
+        <geometry><box><size>0.11 0.04 0.04</size></box></geometry>
+      </collision>
+    </gazebo>
+    <gazebo reference="joint3">
+      <visual>
+        <geometry><box><size>0.096 0.04 0.04</size></box></geometry>
+        <material>
+          <ambient>0.8 0.8 0.8 1</ambient>
+          <diffuse>0.9 0.9 0.9 1</diffuse>
+        </material>
+      </visual>
+      <collision>
+        <geometry><box><size>0.096 0.04 0.04</size></box></geometry>
+      </collision>
+    </gazebo>
+    <gazebo reference="joint4">
+      <visual>
+        <geometry><box><size>0.096 0.04 0.04</size></box></geometry>
+        <material>
+          <ambient>0.4 0.4 0.4 1</ambient>
+          <diffuse>0.5 0.5 0.5 1</diffuse>
+        </material>
+      </visual>
+      <collision>
+        <geometry><box><size>0.096 0.04 0.04</size></box></geometry>
+      </collision>
+    </gazebo>
+    <gazebo reference="joint5">
+      <visual>
+        <geometry>
+          <cylinder><radius>0.03</radius><length>0.04</length></cylinder>
+        </geometry>
+        <material>
+          <ambient>0.1 0.1 0.1 1</ambient>
+          <diffuse>0.2 0.2 0.2 1</diffuse>
+        </material>
+      </visual>
+      <collision>
+        <geometry>
+          <cylinder><radius>0.03</radius><length>0.04</length></cylinder>
+        </geometry>
+      </collision>
+    </gazebo>
+    <gazebo reference="joint6">
+      <visual>
+        <geometry>
+          <cylinder><radius>0.03</radius><length>0.04</length></cylinder>
+        </geometry>
+        <material>
+          <ambient>0.4 0.4 0.4 1</ambient>
+          <diffuse>0.5 0.5 0.5 1</diffuse>
+        </material>
+      </visual>
+      <collision>
+        <geometry>
+          <cylinder><radius>0.03</radius><length>0.04</length></cylinder>
+        </geometry>
+      </collision>
+    </gazebo>
+    <gazebo reference="joint6_flange">
+      <visual>
+        <geometry>
+          <cylinder><radius>0.025</radius><length>0.02</length></cylinder>
+        </geometry>
+        <material>
+          <ambient>0.1 0.1 0.1 1</ambient>
+          <diffuse>0.2 0.2 0.2 1</diffuse>
+        </material>
+      </visual>
+      <collision>
+        <geometry>
+          <cylinder><radius>0.025</radius><length>0.02</length></cylinder>
+        </geometry>
+      </collision>
+    </gazebo>
+  </xacro:if>
 </robot>
